File: DemoGit.kicad_sch (KiCad schematic)
At the start: 16 parts, among them J1 USB_B_Micro, J2 Conn_Coaxial, SW1 SW_Push, U1 AP2112K-3.3, U2 RFM95W-915S2, U3 ATSAMD21G15A-A

Commit message: feat(sch): agrega display e-ink U4 al esquematico
Parts:
- added U4: Waveshare_epaper, Package_QFP:LQFP-100_14x14mm_P0.5mm, symbol E_Ink_Display:E_ink_display
Connections:
- net 3V3: now also U4.8 (VCC)
- net CLK: now also U4.5 (SPLCLK)
- net COPI: now also U4.6 (SPLDIN)
- net GND: now also U4.7 (GND)
